Commit message: gotowe

File: install/prosty_robot_description/share/prosty_robot_description/urdf/prosty_robot.xacro (robot description, xacro)
@@ -2,5 +2,5 @@
 <robot name="prosty_robot" xmlns:xacro="http://www.ros.org/wiki/xacro">
 <xacro:include filename="$(find prosty_robot_description)/urdf/materials.xacro" />
-<xacro:include filename="$(find prosty_robot_description)/urdf/prosty_robot.trans" />
+<xacro:include filename="$(find prosty_robot_description)/urdf/prosty_robot_control.xacro" />
 <xacro:include filename="$(find prosty_robot_description)/urdf/prosty_robot.gazebo" />
 <link name="base_link">
@@ -94,5 +94,5 @@
   <parent link="base_link"/>
   <child link="right_wheel_1"/>
-  <axis xyz="1.0 0.0 0.0"/>
+  <axis xyz="-1.0 0.0 0.0"/>
 </joint>
 <joint name="caster_wheel_joint" type="fixed">
